Commit message: test

File: description/wheel_chair_robot/urdf/wheel_chair_robot.urdf (robot description, URDF)
Before this commit: robot wheel_chair_robot, 7 links, 6 joints
Links:
- removed link imu_link
- added link imu_base, mass 0.00066052; collision mesh filename=package://wheel_chair_robot/meshes/imu_link.STL; visual mesh filename=package://wheel_chair_robot/meshes/imu_link.STL
Joints:
- joint imu_joint: child imu_link -> imu_base
