Commit message: test

File: description/description/urdf/description.urdf (robot description, URDF)
Before this commit: robot description, 6 links, 5 joints
Links:
- added link base_footprint
Joints:
- added joint base_joint: type fixed, parent base_footprint, child base_link, origin xyz=0.0 0.0 0 rpy=0 0 -1.57
- joint lidar_joint: origin xyz=0.0042092 0.080995 0.1732 rpy=3.1416 0 0 -> xyz=0.0042092 0.080995 0.1732 rpy=0 -3.14 1.57

File: description/wheel_chair_robot/urdf/wheel_chair_robot.urdf (robot description, URDF)
Before this commit: robot wheel_chair_robot, 7 links, 6 joints
Joints:
- joint lidar_joint: origin xyz=-0.002 0.079323 0.24026 rpy=0 -3.14 1.57 -> xyz=-0.002 0.079323 0.24026 rpy=0 3.14 1.57

Commit message: 2021.05.23

File: description/description/urdf/description.urdf (robot description, URDF)
Before this commit: robot description, 7 links, 6 joints
Links:
- removed link imu_link
- added link imu_base, mass 0.000942; collision mesh filename=package://description/meshes/imu_link.STL; visual mesh filename=package://description/meshes/imu_link.STL
Joints:
- joint imu_joint: child imu_link -> imu_base; origin xyz=0.0063942 0.10863 0.040861 rpy=3.1416 0 -1.5708 -> xyz=0.0063942 0.10863 0.040861 rpy=0 0 -1.5708
- joint lidar_joint: origin xyz=0.0042092 0.080995 0.1732 rpy=0 -3.14 1.57 -> xyz=0.0042092 0.080995 0.1732 rpy=3.14 -3.14 1.57

Commit message: 2021.05.31_gazebo

File: description/description/urdf/description.urdf (robot description, URDF)
Before this commit: robot description, 7 links, 6 joints
Joints:
- joint lidar_joint: origin xyz=0.0042092 0.080995 0.1732 rpy=3.14 -3.14 1.57 -> xyz=0.0042092 0.080995 0.1932 rpy=3.14 -3.14 1.57

Commit message: 2021.06.04_CV_start

File: description/description/urdf/description.urdf (robot description, URDF)
Before this commit: robot description, 7 links, 6 joints
Links:
- added link usb_cam
Joints:
- added joint cam_joint: type fixed, parent lidar_link, child usb_cam, origin xyz=0.0 0.0 0 rpy=0 0 0
