Commit message: 2021.06.05_final

File: description/description_Final/urdf/description_Final.urdf (robot description, URDF)
Before this commit: robot description_Final, 6 links, 5 joints
Links:
- added link base_footprint
Joints:
- added joint base_joint: type fixed, parent base_footprint, child base_link, origin xyz=0.0 0.0 0 rpy=0 0 -1.57
- joint lidar_joint: origin xyz=-0.002 0.079323 0.22748 rpy=3.1416 0 0 -> xyz=-0.002 0.079323 0.24748 rpy=3.14 -3.14 1.57
